Commit message: Vectorized Env wrapper

File: uqslam/models/pioneer3at/model.xacro (robot description, xacro)
@@ -1,13 +1,13 @@
-<?xml version="1.0" ?>
-<!-- =================================================================================== -->
-<!-- |    This document was autogenerated by xacro from model.xacro                    | -->
-<!-- |    EDITING THIS FILE BY HAND IS NOT RECOMMENDED                                 | -->
-<!-- =================================================================================== -->
+<?xml version="1.0"?>
 <!-- ===== Xacro Macro Header ===== -->
 <!-- arguments="prefix namespace collide_bitmask visible" -->
-<sdf version="1.7">
-  <model name="robot1pioneer3at">
+<sdf version='1.7' xmlns:xacro="http://www.ros.org/wiki/xacro">
+  <xacro:arg name="prefix" default="robot1" />
+  <xacro:arg name="namespace" default="robot1_ns" />
+  <xacro:arg name="collide_bitmask" default="0x01" />
+  <xacro:arg name="visible" default="false" />
+  <model name='$(arg prefix)pioneer3at'>
     <!-- ========== Base Link ========== -->
-    <link name="robot1base_link">
+    <link name='$(arg prefix)base_link'>
       <inertial>
         <pose>-0.000108 0 0.172396 0 -0 0</pose>
@@ -23,5 +23,5 @@
       </inertial>
       <!-- Collisions -->
-      <collision name="robot1base_link_collision">
+      <collision name='$(arg prefix)base_link_collision'>
         <pose>0 0 0.177 0 -0 0</pose>
         <geometry>
@@ -33,13 +33,13 @@
         <surface>
           <contact>
-            <collide_bitmask>0x01</collide_bitmask>
-            <ode/>
-          </contact>
-          <friction>
-            <ode/>
-          </friction>
-        </surface>
-      </collision>
-      <collision name="robot1base_link_fixed_joint_lump__back_sonar_collision_1">
+            <collide_bitmask>$(arg collide_bitmask)</collide_bitmask>
+            <ode />
+          </contact>
+          <friction>
+            <ode />
+          </friction>
+        </surface>
+      </collision>
+      <collision name='$(arg prefix)base_link_fixed_joint_lump__back_sonar_collision_1'>
         <pose>-0.187 0 0.247 0 -0 0</pose>
         <geometry>
@@ -50,13 +50,13 @@
         <surface>
           <contact>
-            <collide_bitmask>0x01</collide_bitmask>
-            <ode/>
-          </contact>
-          <friction>
-            <ode/>
-          </friction>
-        </surface>
-      </collision>
-      <collision name="robot1base_link_fixed_joint_lump__front_sonar_collision_2">
+            <collide_bitmask>$(arg collide_bitmask)</collide_bitmask>
+            <ode />
+          </contact>
+          <friction>
+            <ode />
+          </friction>
+        </surface>
+      </collision>
+      <collision name='$(arg prefix)base_link_fixed_joint_lump__front_sonar_collision_2'>
         <pose>0.193 0 0.25 0 -0 0</pose>
         <geometry>
@@ -67,13 +67,13 @@
         <surface>
           <contact>
-            <collide_bitmask>0x01</collide_bitmask>
-            <ode/>
-          </contact>
-          <friction>
-            <ode/>
-          </friction>
-        </surface>
-      </collision>
-      <collision name="robot1base_link_fixed_joint_lump__p3at_front_left_axle_collision_3">
+            <collide_bitmask>$(arg collide_bitmask)</collide_bitmask>
+            <ode />
+          </contact>
+          <friction>
+            <ode />
+          </friction>
+        </surface>
+      </collision>
+      <collision name='$(arg prefix)base_link_fixed_joint_lump__p3at_front_left_axle_collision_3'>
         <pose>0.135 0.156 0.111 0 -0 0</pose>
         <geometry>
@@ -84,13 +84,13 @@
         <surface>
           <contact>
-            <collide_bitmask>0x01</collide_bitmask>
-            <ode/>
-          </contact>
-          <friction>
-            <ode/>
-          </friction>
-        </surface>
-      </collision>
-      <collision name="robot1base_link_fixed_joint_lump__p3at_front_left_hub_collision_4">
+            <collide_bitmask>$(arg collide_bitmask)</collide_bitmask>
+            <ode />
+          </contact>
+          <friction>
+            <ode />
+          </friction>
+        </surface>
+      </collision>
+      <collision name='$(arg prefix)base_link_fixed_joint_lump__p3at_front_left_hub_collision_4'>
         <pose>0.135 0.197 0.111 0 -0 0</pose>
         <geometry>
@@ -101,13 +101,13 @@
         <surface>
           <contact>
-            <collide_bitmask>0x01</collide_bitmask>
-            <ode/>
-          </contact>
-          <friction>
-            <ode/>
-          </friction>
-        </surface>
-      </collision>
-      <collision name="robot1base_link_fixed_joint_lump__p3at_front_right_axle_collision_5">
+            <collide_bitmask>$(arg collide_bitmask)</collide_bitmask>
+            <ode />
+          </contact>
+          <friction>
+            <ode />
+          </friction>
+        </surface>
+      </collision>
+      <collision name='$(arg prefix)base_link_fixed_joint_lump__p3at_front_right_axle_collision_5'>
         <pose>0.135 -0.156 0.111 0 -0 0</pose>
         <geometry>
@@ -118,13 +118,13 @@
         <surface>
           <contact>
-            <collide_bitmask>0x01</collide_bitmask>
-            <ode/>
-          </contact>
-          <friction>
-            <ode/>
-          </friction>
-        </surface>
-      </collision>
-      <collision name="robot1base_link_fixed_joint_lump__p3at_front_right_hub_collision_6">
+            <collide_bitmask>$(arg collide_bitmask)</collide_bitmask>
+            <ode />
+          </contact>
+          <friction>
+            <ode />
+          </friction>
+        </surface>
+      </collision>
+      <collision name='$(arg prefix)base_link_fixed_joint_lump__p3at_front_right_hub_collision_6'>
         <pose>0.135 -0.197 0.111 0 -0 0</pose>
         <geometry>
@@ -135,13 +135,13 @@
         <surface>
           <contact>
-            <collide_bitmask>0x01</collide_bitmask>
-            <ode/>
-          </contact>
-          <friction>
-            <ode/>
-          </friction>
-        </surface>
-      </collision>
-      <collision name="robot1base_link_fixed_joint_lump__top_plate_collision_7">
+            <collide_bitmask>$(arg collide_bitmask)</collide_bitmask>
+            <ode />
+          </contact>
+          <friction>
+            <ode />
+          </friction>
+        </surface>
+      </collision>
+      <collision name='$(arg prefix)base_link_fixed_joint_lump__top_plate_collision_7'>
         <pose>0.003 0 0.274 0 -0 0</pose>
         <geometry>
@@ -152,13 +152,13 @@
         <surface>
           <contact>
-            <collide_bitmask>0x01</collide_bitmask>
-            <ode/>
-          </contact>
-          <friction>
-            <ode/>
-          </friction>
-        </surface>
-      </collision>
-      <collision name="robot1base_link_fixed_joint_lump__p3at_back_left_axle_collision_8">
+            <collide_bitmask>$(arg collide_bitmask)</collide_bitmask>
+            <ode />
+          </contact>
+          <friction>
+            <ode />
+          </friction>
+        </surface>
+      </collision>
+      <collision name='$(arg prefix)base_link_fixed_joint_lump__p3at_back_left_axle_collision_8'>
         <pose>-0.134 0.156 0.111 0 -0 0</pose>
         <geometry>
@@ -170,13 +170,13 @@
         <surface>
           <contact>
-            <collide_bitmask>0x01</collide_bitmask>
-            <ode/>
-          </contact>
-          <friction>
-            <ode/>
-          </friction>
-        </surface>
-      </collision>
-      <collision name="robot1base_link_fixed_joint_lump__p3at_back_left_hub_collision_9">
+            <collide_bitmask>$(arg collide_bitmask)</collide_bitmask>
+            <ode />
+          </contact>
+          <friction>
+            <ode />
+          </friction>
+        </surface>
+      </collision>
+      <collision name='$(arg prefix)base_link_fixed_joint_lump__p3at_back_left_hub_collision_9'>
         <pose>-0.134 0.197 0.111 0 -0 0</pose>
         <geometry>
@@ -188,13 +188,13 @@
         <surface>
           <contact>
-            <collide_bitmask>0x01</collide_bitmask>
-            <ode/>
-          </contact>
-          <friction>
-            <ode/>
-          </friction>
-        </surface>
-      </collision>
-      <collision name="robot1base_link_fixed_joint_lump__p3at_back_right_axle_collision_10">
+            <collide_bitmask>$(arg collide_bitmask)</collide_bitmask>
+            <ode />
+          </contact>
+          <friction>
+            <ode />
+          </friction>
+        </surface>
+      </collision>
+      <collision name='$(arg prefix)base_link_fixed_joint_lump__p3at_back_right_axle_collision_10'>
         <pose>-0.134 -0.156 0.111 0 -0 0</pose>
         <geometry>
@@ -206,13 +206,13 @@
         <surface>
           <contact>
-            <collide_bitmask>0x01</collide_bitmask>
-            <ode/>
-          </contact>
-          <friction>
-            <ode/>
-          </friction>
-        </surface>
-      </collision>
-      <collision name="robot1base_link_fixed_joint_lump__p3at_back_right_hub_collision_11">
+            <collide_bitmask>$(arg collide_bitmask)</collide_bitmask>
+            <ode />
+          </contact>
+          <friction>
+            <ode />
+          </friction>
+        </surface>
+      </collision>
+      <collision name='$(arg prefix)base_link_fixed_joint_lump__p3at_back_right_hub_collision_11'>
         <pose>-0.134 -0.197 0.111 0 -0 0</pose>
         <geometry>
@@ -224,14 +224,14 @@
         <surface>
           <contact>
-            <collide_bitmask>0x01</collide_bitmask>
-            <ode/>
-          </contact>
-          <friction>
-            <ode/>
+            <collide_bitmask>$(arg collide_bitmask)</collide_bitmask>
+            <ode />
+          </contact>
+          <friction>
+            <ode />
           </friction>
         </surface>
       </collision>
       <!-- Visuals -->
-      <visual name="robot1base_link_visual">
+      <visual name='$(arg prefix)base_link_visual'>
         <pose>0 0 0.177 0 -0 0</pose>
         <geometry>
@@ -247,7 +247,7 @@
           </script>
         </material>
-        <visible>false</visible>
-      </visual>
-      <visual name="robot1base_link_fixed_joint_lump__back_sonar_visual_1">
+        <visible>$(arg visible)</visible>
+      </visual>
+      <visual name='$(arg prefix)base_link_fixed_joint_lump__back_sonar_visual_1'>
         <pose>-0.187 0 0.247 0 -0 0</pose>
         <geometry>
@@ -263,7 +263,7 @@
           </script>
         </material>
-        <visible>false</visible>
-      </visual>
-      <visual name="robot1base_link_fixed_joint_lump__front_sonar_visual_2">
+        <visible>$(arg visible)</visible>
+      </visual>
+      <visual name='$(arg prefix)base_link_fixed_joint_lump__front_sonar_visual_2'>
         <pose>0.193 0 0.25 0 -0 0</pose>
         <geometry>
@@ -279,7 +279,7 @@
           </script>
         </material>
-        <visible>false</visible>
-      </visual>
-      <visual name="robot1base_link_fixed_joint_lump__p3at_front_left_axle_visual_3">
+        <visible>$(arg visible)</visible>
+      </visual>
+      <visual name='$(arg prefix)base_link_fixed_joint_lump__p3at_front_left_axle_visual_3'>
         <pose>0.135 0.156 0.111 0 -0 0</pose>
         <geometry>
@@ -295,7 +295,7 @@
           </script>
         </material>
-        <visible>false</visible>
-      </visual>
-      <visual name="robot1base_link_fixed_joint_lump__p3at_front_left_hub_visual_4">
+        <visible>$(arg visible)</visible>
+      </visual>
+      <visual name='$(arg prefix)base_link_fixed_joint_lump__p3at_front_left_hub_visual_4'>
         <pose>0.135 0.197 0.111 0 -0 0</pose>
         <geometry>
@@ -311,7 +311,7 @@
           </script>
         </material>
-        <visible>false</visible>
-      </visual>
-      <visual name="robot1base_link_fixed_joint_lump__p3at_front_right_axle_visual_5">
+        <visible>$(arg visible)</visible>
+      </visual>
+      <visual name='$(arg prefix)base_link_fixed_joint_lump__p3at_front_right_axle_visual_5'>
         <pose>0.135 -0.156 0.111 0 -0 0</pose>
         <geometry>
@@ -327,7 +327,7 @@
           </script>
         </material>
-        <visible>false</visible>
-      </visual>
-      <visual name="robot1base_link_fixed_joint_lump__p3at_front_right_hub_visual_6">
+        <visible>$(arg visible)</visible>
+      </visual>
+      <visual name='$(arg prefix)base_link_fixed_joint_lump__p3at_front_right_hub_visual_6'>
         <pose>0.135 -0.197 0.111 0 -0 0</pose>
         <geometry>
@@ -343,7 +343,7 @@
           </script>
         </material>
-        <visible>false</visible>
-      </visual>
-      <visual name="robot1base_link_fixed_joint_lump__top_plate_visual_7">
+        <visible>$(arg visible)</visible>
+      </visual>
+      <visual name='$(arg prefix)base_link_fixed_joint_lump__top_plate_visual_7'>
         <pose>0.003 0 0.274 0 -0 0</pose>
         <geometry>
@@ -359,7 +359,7 @@
           </script>
         </material>
-        <visible>false</visible>
-      </visual>
-      <visual name="robot1base_link_fixed_joint_lump__p3at_back_left_axle_visual_8">
+        <visible>$(arg visible)</visible>
+      </visual>
+      <visual name='$(arg prefix)base_link_fixed_joint_lump__p3at_back_left_axle_visual_8'>
         <pose>-0.134 0.156 0.111 0 -0 0</pose>
         <geometry>
@@ -375,7 +375,7 @@
           </script>
         </material>
-        <visible>false</visible>
-      </visual>
-      <visual name="robot1base_link_fixed_joint_lump__p3at_back_left_hub_visual_9">
+        <visible>$(arg visible)</visible>
+      </visual>
+      <visual name='$(arg prefix)base_link_fixed_joint_lump__p3at_back_left_hub_visual_9'>
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
File: uqslam/worlds/circuit.xacro (robot description, xacro)
@@ -1,110 +1,108 @@
 <?xml version="1.0"?>
-<robot xmlns:xacro="http://ros.org/wiki/xacro">
-  <xacro:arg name="speedup" default="false"/>
-  <sdf version='1.4'>
-    <world name='default'>
-      <plugin name="gazebo_ros_state" filename="libgazebo_ros_state.so">
-        <ros>
-          <namespace>/demo</namespace>
-          <remapping>model_states:=model_states_demo</remapping>
-          <remapping>link_states:=link_states_demo</remapping>
-        </ros>
-        <update_rate>1.0</update_rate>
-      </plugin>
-      <light name='sun' type='directional'>
-        <cast_shadows>1</cast_shadows>
-        <pose>0 0 10 0 -0 0</pose>
-        <diffuse>0.8 0.8 0.8 1</diffuse>
-        <specular>0.2 0.2 0.2 1</specular>
-        <attenuation>
-          <range>1000</range>
-          <constant>0.9</constant>
-          <linear>0.01</linear>
-          <quadratic>0.001</quadratic>
-        </attenuation>
-        <direction>0.5 0.1 -0.9</direction>
-      </light>
-      <model name='ground_plane'>
-        <static>1</static>
-        <link name='link'>
-          <collision name='collision'>
-            <geometry>
-              <plane>
-                <normal>0 0 1</normal>
-                <size>100 100</size>
-              </plane>
-            </geometry>
-            <surface>
-              <friction>
-                <ode>
-                  <mu>100</mu>
-                  <mu2>50</mu2>
-                </ode>
-              </friction>
-              <bounce/>
-              <contact>
-                <ode/>
-              </contact>
-            </surface>
-            <max_contacts>10</max_contacts>
-          </collision>
-          <visual name='visual'>
-            <cast_shadows>0</cast_shadows>
-            <geometry>
-              <plane>
-                <normal>0 0 1</normal>
-                <size>100 100</size>
-              </plane>
-            </geometry>
-            <material>
-              <script>
-                <uri>file://media/materials/scripts/gazebo.material</uri>
-                <name>Gazebo/Grey</name>
-              </script>
-            </material>
-          </visual>
-          <velocity_decay>
-            <linear>0</linear>
-            <angular>0</angular>
-          </velocity_decay>
-          <self_collide>0</self_collide>
-          <kinematic>0</kinematic>
-          <gravity>1</gravity>
-        </link>
-      </model>
-      <scene>
-        <ambient>0.4 0.4 0.4 1</ambient>
-        <background>0.7 0.7 0.7 1</background>
-        <shadows>0</shadows>
-      </scene>
-      <physics type='ode'>
-        <max_step_size>0.01</max_step_size>
-        <real_time_factor>
-          <xacro:if value="$(arg speedup)">0</xacro:if>
-          <xacro:unless value="$(arg speedup)">1</xacro:unless>
-        </real_time_factor>
-        <real_time_update_rate>
-          <xacro:if value="$(arg speedup)">0</xacro:if>
-          <xacro:unless value="$(arg speedup)">100</xacro:unless>
-        </real_time_update_rate>
-        <gravity>0 0 -9.8</gravity>
-      </physics>
-      <state world_name='default'>
-        <sim_time>0 0</sim_time>
-        <real_time>0 0</real_time>
-        <wall_time>0 0</wall_time>
-      </state>
-      <gui fullscreen='0'>
-        <camera name='user_camera'>
-          <pose>2.6 -1.69 12.2 0 1.56 3.14</pose>
-          <view_controller>orbit</view_controller>
-        </camera>
-      </gui>
-      <!-- A simple circuit -->
-      <include>
-        <uri>model://Circuit_ql_1</uri>
-        <pose>2.4 -2.1 0 0 0 0</pose>
-      </include>
-    </world>
-  </sdf>
-</robot>
+<sdf version='1.4' xmlns:xacro="http://ros.org/wiki/xacro">
+  <xacro:arg name="speedup" default="false" />
+  <world name='default'>
+    <plugin name="gazebo_ros_state" filename="libgazebo_ros_state.so">
+      <ros>
+        <namespace>/demo</namespace>
+        <remapping>model_states:=model_states_demo</remapping>
+        <remapping>link_states:=link_states_demo</remapping>
+      </ros>
+      <update_rate>1.0</update_rate>
+    </plugin>
+    <light name='sun' type='directional'>
+      <cast_shadows>1</cast_shadows>
+      <pose>0 0 10 0 -0 0</pose>
+      <diffuse>0.8 0.8 0.8 1</diffuse>
+      <specular>0.2 0.2 0.2 1</specular>
+      <attenuation>
+        <range>1000</range>
+        <constant>0.9</constant>
+        <linear>0.01</linear>
+        <quadratic>0.001</quadratic>
+      </attenuation>
+      <direction>0.5 0.1 -0.9</direction>
+    </light>
+    <model name='ground_plane'>
+      <static>1</static>
+      <link name='link'>
+        <collision name='collision'>
+          <geometry>
+            <plane>
+              <normal>0 0 1</normal>
+              <size>100 100</size>
+            </plane>
+          </geometry>
+          <surface>
+            <friction>
+              <ode>
+                <mu>100</mu>
+                <mu2>50</mu2>
+              </ode>
+            </friction>
+            <bounce />
+            <contact>
+              <ode />
+            </contact>
+          </surface>
+          <max_contacts>10</max_contacts>
+        </collision>
+        <visual name='visual'>
+          <cast_shadows>0</cast_shadows>
+          <geometry>
+            <plane>
+              <normal>0 0 1</normal>
+              <size>100 100</size>
+            </plane>
+          </geometry>
+          <material>
+            <script>
+              <uri>file://media/materials/scripts/gazebo.material</uri>
+              <name>Gazebo/Grey</name>
+            </script>
+          </material>
+        </visual>
+        <velocity_decay>
+          <linear>0</linear>
+          <angular>0</angular>
+        </velocity_decay>
+        <self_collide>0</self_collide>
+        <kinematic>0</kinematic>
+        <gravity>1</gravity>
+      </link>
+    </model>
+    <scene>
+      <ambient>0.4 0.4 0.4 1</ambient>
+      <background>0.7 0.7 0.7 1</background>
+      <shadows>0</shadows>
+    </scene>
+    <physics type='ode'>
+      <max_step_size>0.01</max_step_size>
+      <real_time_factor>
+        <xacro:if value="$(arg speedup)">0</xacro:if>
+        <xacro:unless value="$(arg speedup)">1</xacro:unless>
+      </real_time_factor>
+      <real_time_update_rate>
+        <xacro:if value="$(arg speedup)">0</xacro:if>
+        <xacro:unless value="$(arg speedup)">100</xacro:unless>
+      </real_time_update_rate>
+      <gravity>0 0 -9.8</gravity>
+    </physics>
+    <state world_name='default'>
+      <sim_time>0 0</sim_time>
+      <real_time>0 0</real_time>
+      <wall_time>0 0</wall_time>
+    </state>
+    <gui fullscreen='0'>
+      <camera name='user_camera'>
+        <pose>2.6 -1.69 12.2 0 1.56 3.14</pose>
+        <view_controller>orbit</view_controller>
+      </camera>
+    </gui>
+    <!-- A simple circuit -->
+    <include>
+      <uri>model://Circuit_ql_1</uri>
+      <pose>2.4 -2.1 0 0 0 0</pose>
+    </include>
+  </world>
+</sdf>
